File: ATTAMI-V0.00.brd (EAGLE design)
At the start: 22.8 x 22.9 mm, 24 parts, among them U1 MIC5225, U2 ATTINY85

Commit message: added an npn to bottom layer -WIP
Parts:
- removed U$3: (no value), ohw-logo:OSHW_6X150_NOTEXT
- added Q2: (no value), microbuilder:SOT23-W
- added R5: (no value), adafruit:R0805
- added U$4: (no value), ohw-logo:OSHW_6X150_NOTEXT
Connections:
- new net N$1: Q2.1, R5.2
- net GND: now also Q2.2
- net PB0: now also R5.1
Routing:
- net PB0: track 5.19 -> 11.5 mm
- net N$1: track 0.00 -> 3.35 mm
Other:
- board text removed: "ATtami"
- board text removed: "J2"
Changed lines of the file:
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@@
 <layers>
 <layer number="1" name="Top" color="4" fill="1" visible="yes" active="yes"/>
-<layer number="2" name="Route2" color="1" fill="3" visible="no" active="no"/>
-<layer number="3" name="Route3" color="4" fill="3" visible="no" active="no"/>
-<layer number="4" name="Route4" color="1" fill="4" visible="no" active="no"/>
-<layer number="5" name="Route5" color="4" fill="4" visible="no" active="no"/>
-<layer number="6" name="Route6" color="1" fill="8" visible="no" active="no"/>
-<layer number="7" name="Route7" color="4" fill="8" visible="no" active="no"/>
-<layer number="8" name="Route8" color="1" fill="2" visible="no" active="no"/>
-<layer number="9" name="Route9" color="4" fill="2" visible="no" active="no"/>
-<layer number="10" name="Route10" color="1" fill="7" visible="no" active="no"/>
-<layer number="11" name="Route11" color="4" fill="7" visible="no" active="no"/>
-<layer number="12" name="Route12" color="1" fill="5" visible="no" active="no"/>
-<layer number="13" name="Route13" color="4" fill="5" visible="no" active="no"/>
-<layer number="14" name="Route14" color="1" fill="6" visible="no" active="no"/>
-<layer number="15" name="Route15" color="4" fill="6" visible="no" active="no"/>
 <layer number="16" name="Bottom" color="1" fill="1" visible="yes" active="yes"/>
 <layer number="17" name="Pads" color="2" fill="1" visible="yes" active="yes"/>
@@
 <layer number="23" name="tOrigins" color="15" fill="1" visible="yes" active="yes"/>
 <layer number="24" name="bOrigins" color="15" fill="1" visible="yes" active="yes"/>
-<layer number="25" name="tNames" color="7" fill="1" visible="no" active="yes"/>
-<layer number="26" name="bNames" color="7" fill="1" visible="no" active="yes"/>
-<layer number="27" name="tValues" color="7" fill="1" visible="no" active="yes"/>
-<layer number="28" name="bValues" color="7" fill="1" visible="no" active="yes"/>
+<layer number="25" name="tNames" color="7" fill="1" visible="yes" active="yes"/>
+<layer number="26" name="bNames" color="7" fill="1" visible="yes" active="yes"/>
+<layer number="27" name="tValues" color="7" fill="1" visible="yes" active="yes"/>
+<layer number="28" name="bValues" color="7" fill="1" visible="yes" active="yes"/>
 <layer number="29" name="tStop" color="7" fill="3" visible="no" active="yes"/>
 <layer number="30" name="bStop" color="7" fill="6" visible="no" active="yes"/>
 <layer number="31" name="tCream" color="12" fill="1" visible="no" active="yes"/>
 <layer number="32" name="bCream" color="7" fill="5" visible="no" active="yes"/>
-<layer number="37" name="tTest" color="7" fill="1" visible="no" active="yes"/>
+<layer number="33" name="tFinish" color="6" fill="3" visible="no" active="yes"/>
+<layer number="34" name="bFinish" color="6" fill="6" visible="no" active="yes"/>
+<layer number="36" name="bGlue" color="7" fill="5" visible="no" active="yes"/>
 <layer number="39" name="tKeepout" color="4" fill="11" visible="no" active="yes"/>
 <layer number="40" name="bKeepout" color="1" fill="11" visible="no" active="yes"/>
@@
 <layer number="47" name="Measures" color="7" fill="1" visible="no" active="yes"/>
 <layer number="48" name="Document" color="7" fill="1" visible="no" active="yes"/>
-<layer number="50" name="dxf" color="7" fill="1" visible="no" active="no"/>
+<layer number="49" name="Reference" color="7" fill="1" visible="no" active="yes"/>
 <layer number="51" name="tDocu" color="7" fill="1" visible="yes" active="yes"/>
 <layer number="52" name="bDocu" color="7" fill="1" visible="no" active="yes"/>
-<layer number="53" name="tGND_GNDA" color="7" fill="9" visible="no" active="no"/>
-<layer number="54" name="bGND_GNDA" color="1" fill="9" visible="no" active="no"/>
-<layer number="56" name="wert" color="7" fill="1" visible="no" active="no"/>
 <layer number="91" name="Nets" color="2" fill="1" visible="no" active="no"/>
 <layer number="92" name="Busses" color="1" fill="1" visible="no" active="no"/>
@@
 <layer number="97" name="Info" color="7" fill="1" visible="no" active="no"/>
 <layer number="98" name="Guide" color="6" fill="1" visible="no" active="no"/>
-<layer number="118" name="Rect_Pads" color="7" fill="1" visible="no" active="no"/>
-<layer number="217" name="217bmp" color="18" fill="1" visible="no" active="no"/>
-<layer number="218" name="218bmp" color="19" fill="1" visible="no" active="no"/>
-<layer number="219" name="219bmp" color="20" fill="1" visible="no" active="no"/>
-<layer number="220" name="220bmp" color="21" fill="1" visible="no" active="no"/>
-<layer number="221" name="221bmp" color="22" fill="1" visible="no" active="no"/>
-<layer number="222" name="222bmp" color="23" fill="1" visible="no" active="no"/>
-<layer number="223" name="223bmp" color="24" fill="1" visible="no" active="no"/>
-<layer number="224" name="224bmp" color="25" fill="1" visible="no" active="no"/>
-<layer number="250" name="Descript" color="3" fill="1" visible="no" active="no"/>
-<layer number="251" name="SMDround" color="12" fill="11" visible="no" active="no"/>
 </layers>
 <board>
@@
 <wire x1="22.829840625" y1="22.8602" x2="0" y2="22.8602" width="0" layer="20"/>
 <wire x1="0" y1="22.8602" x2="0" y2="0" width="0" layer="20"/>
-<text x="18.864790625" y="2.510065625" size="1.016" layer="25" rot="R45">VCC</text>
+<text x="18.991790625" y="2.891065625" size="1.016" layer="25" rot="R45">VCC</text>
 <text x="2.9708375" y="7.672909375" size="1.016" layer="25" rot="R60">PB2</text>
 <text x="3.33760625" y="10.141159375" size="1.016" layer="25" rot="R60">PB1</text>
@@
 <wire x1="19.9263" y1="11.320784375" x2="19.9263" y2="11.828784375" width="0.127" layer="21"/>
 <text x="19.423715625" y="15.208471875" size="0.9398" layer="25" rot="R270">BAT</text>
-<text x="21.9459375" y="5.2294875" size="1.143" layer="25" rot="R90">ATtami</text>
-<text x="17.4644375" y="21.6462375" size="1.0668" layer="37" rot="R180">J2</text>
 <wire x1="19.4354625" y1="0.6601" x2="19.6894625" y2="0.6601" width="0.127" layer="21"/>
 <wire x1="19.1830625" y1="0.9685" x2="19.9450625" y2="0.9685" width="0.127" layer="21"/>
@@
 </element>
 <element name="U$1" library="microbuilder" package="MOUNTINGHOLE_2.0_PLATED" value="MOUNTINGHOLE2.0" x="2.54" y="20.32" smashed="yes" rot="R270"/>
-<element name="S1" library="SparkFun-Electromechanical" package="TACTILE-SWITCH-1101NE" value="SWITCH-MOMENTARY-2-SMD-1101NE" x="11.2014" y="1.8034" smashed="yes" rot="R180">
-<attribute name="NAME" x="12.4234" y="4.8834" size="1.016" layer="37" rot="R180"/>
-</element>
+<element name="S1" library="SparkFun-Electromechanical" package="TACTILE-SWITCH-1101NE" value="SWITCH-MOMENTARY-2-SMD-1101NE" x="11.2014" y="1.8034" smashed="yes" rot="R180"/>
 <element name="USB" library="yair_r" package="USB-MICRO-ALIEXPRESS" value="MICRO-USB_ALIEXPRESS" x="10.873740625" y="20.1803" smashed="yes" rot="R180"/>
 <element name="U$2" library="microbuilder" package="MOUNTINGHOLE_2.0_PLATED" value="MOUNTINGHOLE2.0" x="20.32" y="20.32" smashed="yes"/>
-<element name="J2" library="microbuilder" package="1X02_ROUND" value="" x="21.59" y="12.7" smashed="yes" rot="R270">
-<attribute name="NAME" x="20.843240625" y="8.666478125" size="1.27" layer="37" ratio="10"/>
-</element>
-<element name="J3" library="microbuilder" package="1X02_ROUND" value="" x="21.59" y="2.54" smashed="yes" rot="R270">
-<attribute name="NAME" x="20.77211875" y="5.6286375" size="1.27" layer="37" ratio="10"/>
-</element>
+<element name="J2" library="microbuilder" package="1X02_ROUND" value="" x="21.59" y="12.7" smashed="yes" rot="R270"/>
+<element name="J3" library="microbuilder" package="1X02_ROUND" value="" x="21.59" y="2.54" smashed="yes" rot="R270"/>
 <element name="J1" library="microbuilder" package="1X07_ROUND" value="" x="1.27" y="8.89" smashed="yes" rot="R270">
 <attribute name="VALUE" x="-1.905" y="17.78" size="0.4064" layer="27" ratio="10" rot="R270"/>
@@
 <attribute name="VALUE" x="2.7178" y="13.7922" size="1.27" layer="27"/>
 </element>
-<element name="U$3" library="ohw-logo" package="OSHW_6X150_NOTEXT" value="" x="10.668" y="7.112" rot="R90"/>
+<element name="U$4" library="ohw-logo" package="OSHW_6X150_NOTEXT" value="" x="22.352" y="5.842" rot="R90"/>
+<element name="R5" library="adafruit" package="R0805" value="" x="5.461" y="8.001" smashed="yes" rot="MR250">
+<attribute name="VALUE" x="7.34851875" y="9.498903125" size="1.27" layer="28" rot="MR250"/>
+</element>
+<element name="Q2" library="microbuilder" package="SOT23-W" value="" x="6.858" y="2.413" rot="MR180"/>
 </elements>
 <signals>
@@
 <wire x1="9.8298" y1="10.8966" x2="12.227559375" y2="11.1277375" width="0.4064" layer="1" curve="29.414871"/>
 <contactref element="J1" pad="1"/>
-<via x="5.30351875" y="4.119878125" extent="1-16" drill="0.6"/>
+<via x="4.54151875" y="4.246878125" extent="1-16" drill="0.6"/>
 <contactref element="SJ1" pad="1"/>
 <contactref element="COIN_CELL_(-)" pad="1"/>
@@
 <wire x1="9.4107" y1="18.161" x2="9.573740625" y2="18.2553" width="0.2032" layer="1"/>
 <wire x1="4.1275" y1="17.0053" x2="3.9878" y2="16.9672" width="0.2032" layer="1"/>
+<contactref element="Q2" pad="2"/>
 </signal>
 <signal name="PB3">
@@
 <wire x1="1.27" y1="13.97" x2="4.826" y2="11.176" width="0.4064" layer="1"/>
 <wire x1="4.826" y1="11.176" x2="5.496559375" y2="11.1277375" width="0.4064" layer="1"/>
+<contactref element="R5" pad="1"/>
+<wire x1="5.11898125" y1="8.940690625" x2="1.27" y2="13.97" width="0.3048" layer="16"/>
 </signal>
 <signal name="PB2">
@@
 <wire x1="19.550940625" y1="16.637" x2="19.7257875" y2="16.462153125" width="0.4064" layer="1"/>
 </signal>
+<signal name="N$1">
+<contactref element="R5" pad="2"/>
+<contactref element="Q2" pad="1"/>
+<wire x1="5.803021875" y1="7.06130625" x2="5.758" y2="3.713" width="0.3048" layer="16"/>
+</signal>
 </signals>
