File: ATTAMI-V0.00.sch (EAGLE design)
At the start: 23 parts, among them U1 MIC5225, U2 ATTINY85

Commit message: added an npn to bottom layer -WIP
Parts:
- added Q2: (no value), microbuilder:TRANSISTOR_NPNWAVE
- added R5: (no value), adafruit:R-US_R0805
Connections:
- new net N$1: Q2.B, R5.2
- net GND: now also Q2.E
- net PB0: now also R5.1
Changed lines of the file:
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@@
 <part name="COIN_CELL_(+)" library="adafruit" deviceset="PINHD-1X1" device="CB"/>
 <part name="COIN_CELL_(-)" library="adafruit" deviceset="PINHD-1X1" device="CB"/>
+<part name="R5" library="adafruit" deviceset="R-US_" device="R0805"/>
+<part name="GND7" library="SparkFun" deviceset="GND" device=""/>
+<part name="Q2" library="microbuilder" deviceset="TRANSISTOR_NPN" device="WAVE"/>
 </parts>
 <sheets>
@@
 <attribute name="VALUE" x="115.57" y="134.62" size="1.778" layer="96"/>
 </instance>
+<instance part="R5" gate="G$1" x="190.5" y="149.86"/>
+<instance part="GND7" gate="1" x="203.2" y="139.7"/>
+<instance part="Q2" gate="G$1" x="203.2" y="149.86"/>
 </instances>
 <busses>
@@
 <wire x1="139.7" y1="96.52" x2="142.24" y2="96.52" width="0.1524" layer="91"/>
 </segment>
+<segment>
+<pinref part="GND7" gate="1" pin="GND"/>
+<pinref part="Q2" gate="G$1" pin="E"/>
+<wire x1="203.2" y1="142.24" x2="203.2" y2="144.78" width="0.1524" layer="91"/>
+</segment>
 </net>
 <net name="PB3" class="0">
@@
 <segment>
 <pinref part="U2" gate="G$1" pin="PB0(MOSI)"/>
-<wire x1="231.14" y1="127" x2="175.26" y2="127" width="0.1524" layer="91"/>
+<wire x1="231.14" y1="127" x2="180.34" y2="127" width="0.1524" layer="91"/>
 <pinref part="J1" gate="A" pin="2"/>
+<pinref part="R5" gate="G$1" pin="1"/>
+<wire x1="180.34" y1="127" x2="175.26" y2="127" width="0.1524" layer="91"/>
+<wire x1="185.42" y1="149.86" x2="180.34" y2="149.86" width="0.1524" layer="91"/>
+<wire x1="180.34" y1="149.86" x2="180.34" y2="127" width="0.1524" layer="91"/>
+<junction x="180.34" y="127"/>
 </segment>
 </net>
@@
 </segment>
 </net>
+<net name="N$1" class="0">
+<segment>
+<pinref part="R5" gate="G$1" pin="2"/>
+<wire x1="195.58" y1="149.86" x2="198.12" y2="149.86" width="0.1524" layer="91"/>
+<pinref part="Q2" gate="G$1" pin="B"/>
+</segment>
+</net>
